File: KiCad/schematic_diagram/schematic_diagram.sch (KiCad schematic (older format))
At the start: 21 parts, among them J1 PROGRAM, Q1 PN2222A, Q2 PN2222A, Q3 Q_PMOS_DSG, U1 STM32F030F4Px, U2 w25q64fw, Y1 8MHz

Commit message: KiCad scheme updated
Parts:
- R0: value R -> 10k
Connections:
- wire segments 113 -> 111
Other:
- moved on the sheet: R0
Changed lines of the file:
@@
 	1    0    0    -1
 $EndComp
-Wire Wire Line
-	3850 6750 3850 6650
 Connection ~ 3850 6650
 Entry Wire Line
@@
 L Device:R R0
 U 1 1 5F5F858D
-P 2100 1750
-F 0 "R0" V 1893 1750 50  0000 C CNN
-F 1 "R" V 1984 1750 50  0000 C CNN
-F 2 "" V 2030 1750 50  0001 C CNN
-F 3 "~" H 2100 1750 50  0001 C CNN
-	1    2100 1750
+P 2100 1950
+F 0 "R0" V 1893 1950 50  0000 C CNN
+F 1 "10k" V 1984 1950 50  0000 C CNN
+F 2 "" V 2030 1950 50  0001 C CNN
+F 3 "~" H 2100 1950 50  0001 C CNN
+	1    2100 1950
 	0    1    1    0
 $EndComp
@@
 L power:GND #PWR0105
 U 1 1 5F5FCE41
-P 1550 1900
-F 0 "#PWR0105" H 1550 1650 50  0001 C CNN
-F 1 "GND" H 1555 1727 50  0000 C CNN
-F 2 "" H 1550 1900 50  0001 C CNN
-F 3 "" H 1550 1900 50  0001 C CNN
-	1    1550 1900
-	1    0    0    -1
+P 1600 1950
+F 0 "#PWR0105" H 1600 1700 50  0001 C CNN
+F 1 "GND" H 1605 1777 50  0000 C CNN
+F 2 "" H 1600 1950 50  0001 C CNN
+F 3 "" H 1600 1950 50  0001 C CNN
+	1    1600 1950
+	0    1    1    0
 $EndComp
 Wire Wire Line
-	2600 1750 2250 1750
+	2600 1950 2250 1950
 Wire Wire Line
-	1950 1750 1550 1750
-Wire Wire Line
-	1550 1750 1550 1900
-NoConn ~ 2600 1950
+	1950 1950 1600 1950
 Text Notes 3650 2750 0    50   Italic 0
 PRG
@@
 Wire Wire Line
 	5750 4050 5750 4250
+Connection ~ 5750 4250
+Wire Wire Line
+	5750 4250 5300 4250
+NoConn ~ 2600 1750
 Wire Bus Line
 	7650 900  7650 4150
@@
 Wire Bus Line
 	4500 900  4500 6950
-Connection ~ 5750 4250
-Wire Wire Line
-	5750 4250 5300 4250
 $EndSCHEMATC

Commit message: Schema updated
Parts:
- removed D2: D, symbol Device:D
- removed Q3: Q_PMOS_DSG, symbol Device:Q_PMOS_DSG
- added D2: SS12, symbol Device:D_Schottky
- added D3: 1N4148.133, symbol Device:D
- added Q3: AO3401A, Package_TO_SOT_SMD:SOT-23, symbol Transistor_FET:AO3401A
- C0: value CP -> 100uF
- R3: value 1k..5k1 -> 1k
- R4: value 10k..100k -> 100k
- R5: value 4k7 -> 10k
Connections:
- wire segments 111 -> 112
Other:
- note added: "BACKUPED_POWER_SUPPLY"
- note added: "Note: PA10 is used for both: LCD reset and power failure detection. During the start the pin behavour is changed."
- note added: "POWER FAILURE DETECTION"
- note added: "POWER SUPPLY (LCD, MEM)"
- note removed: "BACKUP_POWER"
- note removed: "MAIN_POWER"
- note removed: "RESET_LCD & READ POWER FAILURE"
Changed lines of the file:
@@
 encoding utf-8
 Sheet 1 1
-Title ""
-Date ""
-Rev ""
+Title "FUNNY WATCH"
+Date "2020-08-31"
+Rev "1"
 Comp ""
 Comment1 ""
@@
 	2200 5750 2100 5750
 $Comp
-L Device:Q_PMOS_DSG Q3
-U 1 1 5F56BEB5
-P 2950 6000
-F 0 "Q3" H 3155 6046 50  0000 L CNN
-F 1 "Q_PMOS_DSG" H 3155 5955 50  0000 L CNN
-F 2 "" H 3150 6100 50  0001 C CNN
-F 3 "~" H 2950 6000 50  0001 C CNN
-	1    2950 6000
-	1    0    0    -1
-$EndComp
-$Comp
 L Device:CP C0
 U 1 1 5F568D12
 P 3850 5700
 F 0 "C0" H 3968 5746 50  0000 L CNN
-F 1 "CP" H 3968 5655 50  0000 L CNN
+F 1 "100uF" H 3968 5655 50  0000 L CNN
 F 2 "" H 3888 5550 50  0001 C CNN
 F 3 "~" H 3850 5700 50  0001 C CNN
@@
 P 2500 6350
 F 0 "R5" H 2570 6396 50  0000 L CNN
-F 1 "4k7" H 2570 6305 50  0000 L CNN
+F 1 "10k" H 2570 6305 50  0000 L CNN
 F 2 "" V 2430 6350 50  0001 C CNN
 F 3 "~" H 2500 6350 50  0001 C CNN
@@
 P 1800 5750
 F 0 "R3" V 1593 5750 50  0000 C CNN
-F 1 "1k..5k1" V 1684 5750 50  0000 C CNN
+F 1 "1k" V 1684 5750 50  0000 C CNN
 F 2 "" V 1730 5750 50  0001 C CNN
 F 3 "~" H 1800 5750 50  0001 C CNN
@@
 P 2100 6350
 F 0 "R4" H 2170 6396 50  0000 L CNN
-F 1 "10k..100k" H 2170 6305 50  0000 L CNN
+F 1 "100k" H 2170 6305 50  0000 L CNN
 F 2 "" V 2030 6350 50  0001 C CNN
 F 3 "~" H 2100 6350 50  0001 C CNN
@@
 	1    0    0    -1
 $EndComp
-$Comp
-L Device:D D2
-U 1 1 5F560D66
-P 1800 5400
-F 0 "D2" H 1800 5183 50  0000 C CNN
-F 1 "D" H 1800 5274 50  0000 C CNN
-F 2 "" H 1800 5400 50  0001 C CNN
-F 3 "~" H 1800 5400 50  0001 C CNN
-	1    1800 5400
-	-1   0    0    1
-$EndComp
-Wire Wire Line
-	1450 6500 1450 7050
+Wire Wire Line
+	1450 6500 1450 6700
 Entry Wire Line
 	4400 7050 4500 6950
@@
 	1100 5050 1100 5400
 Text Notes 3650 5050 2    50   Italic 0
-MAIN_POWER
-Text Notes 3700 5400 2    50   Italic 0
-BACKUP_POWER
+POWER SUPPLY (LCD, MEM)
+Text Notes 3800 5400 2    50   Italic 0
+BACKUPED_POWER_SUPPLY
 $Comp
 L Device:R R0
@@
 PRG
 Text Notes 2150 7050 0    50   Italic 0
-RESET_LCD & READ POWER FAILURE
+POWER FAILURE DETECTION
 Wire Wire Line
 	5950 4050 5750 4050
@@
 	5750 4250 5300 4250
 NoConn ~ 2600 1750
+$Comp
+L Transistor_FET:AO3401A Q3
+U 1 1 5F4CF8F5
+P 2950 6000
+F 0 "Q3" H 3155 6046 50  0000 L CNN
+F 1 "AO3401A" H 3155 5955 50  0000 L CNN
+F 2 "Package_TO_SOT_SMD:SOT-23" H 3150 5925 50  0001 L CIN
+F 3 "http://www.aosmd.com/pdfs/datasheet/AO3401A.pdf" H 2950 6000 50  0001 L CNN
+	1    2950 6000
+	1    0    0    -1
+$EndComp
+$Comp
+L Device:D D3
+U 1 1 5F4D28EC
+P 1450 6850
+F 0 "D3" V 1496 6770 50  0000 R CNN
+F 1 "1N4148.133" V 1405 6770 50  0000 R CNN
+F 2 "" H 1450 6850 50  0001 C CNN
+F 3 "~" H 1450 6850 50  0001 C CNN
+	1    1450 6850
+	0    -1   -1   0
+$EndComp
+Wire Wire Line
+	1450 7000 1450 7050
+$Comp
+L Device:D_Schottky D2
+U 1 1 5F4E0C7D
+P 1800 5400
+F 0 "D2" H 1800 5183 50  0000 C CNN
+F 1 "SS12" H 1800 5274 50  0000 C CNN
+F 2 "" H 1800 5400 50  0001 C CNN
+F 3 "~" H 1800 5400 50  0001 C CNN
+	1    1800 5400
+	-1   0    0    1
+$EndComp
+Text Notes 6200 6000 0    50   ~ 0
+Note: PA10 is used for both: LCD reset and power failure detection. During the start the pin behavour is changed.
 Wire Bus Line
 	7650 900  7650 4150
