File: KiCad/schematic_diagram/schematic_diagram_v1.sch (KiCad schematic (older format))
At the start: 22 parts, among them J1 PROGRAM, Q1 PN2222A, Q2 PN2222A, Q3 AO3401A, U1 STM32F030F4Px, U2 w25q64fw, Y1 8MHz

Commit message: PCB updated, schema v2 added
Connections:
- net a13: now also J1.2 (Pin_2); no longer J1.1 (Pin_1)
- net a14: now also J1.1 (Pin_1); no longer J1.2 (Pin_2)
Changed lines of the file:
@@
 	8350 1300 7750 1300
 Text Label 7750 1200 0    50   ~ 0
+a14
+Text Label 7750 1300 0    50   ~ 0
 a13
-Text Label 7750 1300 0    50   ~ 0
-a14
 $Comp
 L Connector_Generic:Conn_01x03 J1
