File: KiCad/schematic_diagram/schematic_diagram_v2.sch (KiCad schematic (older format))
At the start: 22 parts, among them J1 PROGRAM, Q1 PN2222A, Q2 PN2222A, Q3 AO3401A, U1 STM32F030F4Px, U2 w25q64fw, Y1 8MHz

Commit message: 3
Parts:
- added to_RX, to_TX: TestPoint_Small, symbol Connector:TestPoint_Small
- J1: value PROGRAM -> MCU PROGRAMMING
Connections:
- net a2: now also to_RX.1
- net a3: now also to_TX.1
Other:
- note added: "GND"
- note added: "SPI Memory programming"
- note added: "SWCLK"
- note added: "SWDIO"
- note added: "USART_RX"
- note added: "USART_TX"
Changed lines of the file:
@@
 P 8550 1300
 F 0 "J1" H 8630 1342 50  0000 L CNN
-F 1 "PROGRAM" H 8630 1251 50  0000 L CNN
+F 1 "MCU PROGRAMMING" H 8630 1251 50  0000 L CNN
 F 2 "" H 8550 1300 50  0001 C CNN
 F 3 "~" H 8550 1300 50  0001 C CNN
@@
 Wire Wire Line
 	2700 4350 4400 4350
+Entry Wire Line
+	7650 3100 7750 3200
+Entry Wire Line
+	7650 3200 7750 3300
+Wire Wire Line
+	7750 3200 8500 3200
+Wire Wire Line
+	7750 3300 8500 3300
 Wire Bus Line
 	7650 900  7650 4150
@@
 Wire Bus Line
 	4500 900  4500 6950
+Text Label 7750 3300 0    50   ~ 0
+a3
+Text Label 7750 3200 0    50   ~ 0
+a2
+Text Notes 8100 3200 0    50   ~ 0
+USART_TX
+Text Notes 8100 3300 0    50   ~ 0
+USART_RX
+$Comp
+L Connector:TestPoint_Small to_TX
+U 1 1 5F56EBC8
+P 8500 3300
+F 0 "to_TX" H 8548 3300 50  0000 L CNN
+F 1 "TestPoint_Small" H 8548 3255 50  0001 L CNN
+F 2 "" H 8700 3300 50  0001 C CNN
+F 3 "~" H 8700 3300 50  0001 C CNN
+	1    8500 3300
+	1    0    0    -1
+$EndComp
+$Comp
+L Connector:TestPoint_Small to_RX
+U 1 1 5F56F5A0
+P 8500 3200
+F 0 "to_RX" H 8548 3200 50  0000 L CNN
+F 1 "TestPoint_Small" H 8548 3155 50  0001 L CNN
+F 2 "" H 8700 3200 50  0001 C CNN
+F 3 "~" H 8700 3200 50  0001 C CNN
+	1    8500 3200
+	1    0    0    -1
+$EndComp
+Text Notes 8800 3300 0    50   ~ 0
+SPI Memory programming
+Text Notes 8050 1300 0    50   ~ 0
+SWDIO
+Text Notes 8050 1200 0    50   ~ 0
+SWCLK
+Text Notes 8050 1400 0    50   ~ 0
+GND
 $EndSCHEMATC
