File: KiCad/schematic_diagram/schematic_diagram_v2.sch (KiCad schematic (older format))
At the start: 24 parts, among them J1 MCU PROGRAMMING, Q1 PN2222A, Q2 PN2222A, Q3 AO3401A, U1 STM32F030F4Px, U2 w25q64fw, Y1 8MHz

Commit message: 8
Parts:
- added D3: SS12, symbol Device:D_Schottky
- R2: value 100k -> 10k
Connections:
- wire segments 117 -> 118
Changed lines of the file:
@@
 P 1100 6350
 F 0 "R2" H 1170 6396 50  0000 L CNN
-F 1 "100k" H 1170 6305 50  0000 L CNN
+F 1 "10k" H 1170 6305 50  0000 L CNN
 F 2 "" V 1030 6350 50  0001 C CNN
 F 3 "~" H 1100 6350 50  0001 C CNN
@@
 Connection ~ 1800 5050
 Wire Wire Line
-	1800 5050 4400 5050
+	1800 5050 2100 5050
 Wire Wire Line
 	1100 6200 1100 5400
@@
 Wire Bus Line
 	4500 900  4500 6950
+$Comp
+L Device:D_Schottky D3
+U 1 1 5F5F7CFF
+P 2250 5050
+F 0 "D3" H 2150 5150 50  0000 C CNN
+F 1 "SS12" H 2100 5250 50  0000 C CNN
+F 2 "" H 2250 5050 50  0001 C CNN
+F 3 "~" H 2250 5050 50  0001 C CNN
+	1    2250 5050
+	-1   0    0    1
+$EndComp
+Wire Wire Line
+	2400 5050 4400 5050
 $EndSCHEMATC

Commit message: clap detector added
Parts:
- added C4: 1000uF, symbol Device:CP
- added C5: 10uF, symbol Device:C
- added C6: 1uF, symbol Device:C
- added D4: SS12, symbol Device:D_Schottky
- added L1: 1000uH, symbol Device:L_Core_Ferrite
- added MK1: DGO4522DD, symbol Device:Microphone
- added R10: 1M, symbol Device:R
- added R11: 220k, symbol Device:R
- added R6: 3k, symbol Device:R
- added R7: 1k, symbol Device:R
- added R8, R9: R, symbol Device:R
- added RV1: 100k, symbol Device:R_POT
- added SW?: SW_Push, symbol Switch:SW_Push
- added U3: LM358, symbol Amplifier_Operational:LM358
- added U4: ATtiny13A-SSU, Package_SO:SOIC-8_3.9x4.9mm_P1.27mm, symbol MCU_Microchip_ATtiny:ATtiny13A-SSU
- renumbered to_RX to to_RX1, to_TX to to_TX1
Connections:
- net labels added: b3
- wire segments 118 -> 167
Other:
- note added: "CLAP DETECTION UNIT (LCD BACKLIGHT CONTROL)"
- note added: "POWER CONTROL UNIT"
- note added: "backuped power supply"
- note added: "power failure detection"
- note added: "power supply (LCD, MEM)"
- note removed: "BACKUPED_POWER_SUPPLY"
- note removed: "POWER FAILURE DETECTION"
- note removed: "POWER SUPPLY (LCD, MEM)"
- moved on the sheet: U2

Commit message: kicad schemes update
Parts:
- removed BT1: CR2035, symbol Device:Battery_Cell
- added Cbak: Ionistor, symbol ez_library:Ionistor
- U4: symbol MCU_Microchip_ATtiny:ATtiny13A-SSU -> schematic_diagram_v2-rescue:ATtiny13A-SSU-MCU_Microchip_ATtiny
Changed lines of the file:
@@
 EESchema Schematic File Version 4
 LIBS:schematic_diagram_v2-cache
-EELAYER 26 0
+EELAYER 29 0
 EELAYER END
 $Descr A4 11693 8268
@@
 	1    0    0    -1
 $EndComp
-Connection ~ 3050 6650
 Wire Wire Line
 	3850 6650 3850 5850
-Wire Wire Line
-	3050 6650 3850 6650
 Connection ~ 3050 5400
 Wire Wire Line
@@
 Wire Wire Line
 	2500 5400 3050 5400
-Wire Wire Line
-	2500 6650 3050 6650
 Connection ~ 2500 6650
 Wire Wire Line
 	2500 6500 2500 6650
-Wire Wire Line
-	3050 6650 3050 6500
 Wire Wire Line
 	2100 6650 2500 6650
@@
 F 3 "~" H 3850 5700 50  0001 C CNN
 	1    3850 5700
-	1    0    0    -1
-$EndComp
-$Comp
-L Device:Battery_Cell BT1
-U 1 1 5F568343
-P 3050 6400
-F 0 "BT1" H 3168 6496 50  0000 L CNN
-F 1 "CR2035" H 3168 6405 50  0000 L CNN
-F 2 "" V 3050 6460 50  0001 C CNN
-F 3 "~" V 3050 6460 50  0001 C CNN
-	1    3050 6400
 	1    0    0    -1
 $EndComp
@@
 	5750 4800 6650 4800
 $Comp
-L MCU_Microchip_ATtiny:ATtiny13A-SSU U4
+L schematic_diagram_v2-rescue:ATtiny13A-SSU-MCU_Microchip_ATtiny U4
 U 1 1 5F9AB5F9
 P 10400 5450
@@
 Wire Wire Line
 	9100 5450 9800 5450
-Wire Bus Line
-	7650 900  7650 4050
-Wire Bus Line
-	5200 900  5200 4050
-Wire Bus Line
-	4500 900  4500 6950
 $Comp
 L Switch:SW_Push SW?
@@
 	1    0    0    -1
 $EndComp
+$Comp
+L ez_library:Ionistor Cbak
+U 1 1 65B75F4C
+P 3050 6400
+F 0 "Cbak" H 3236 6446 50  0000 L CNN
+F 1 "Ionistor" H 3236 6355 50  0000 L CNN
+F 2 "" H 3088 6250 50  0001 C CNN
+F 3 "" H 3050 6400 50  0001 C CNN
+	1    3050 6400
+	1    0    0    -1
+$EndComp
+Wire Wire Line
+	2500 6650 3050 6650
+Wire Wire Line
+	3050 6600 3050 6650
+Wire Bus Line
+	7650 900  7650 4050
+Wire Bus Line
+	5200 900  5200 4050
+Wire Bus Line
+	4500 900  4500 6950
+Connection ~ 3050 6650
+Wire Wire Line
+	3050 6650 3850 6650
 $EndSCHEMATC
